File: groovy/groovy.brd (EAGLE design)
At the start: 160 x 100 mm, 6 parts, among them J1 USB_MICRO, U1 AP7312-1833

Commit message: add charger
Connections:
- new net N$1: C1.2, U1.5
- net VCC: no longer C1.2, U1.5
Changed lines of the file:
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@@
 <?xml version="1.0" encoding="utf-8"?>
 <!DOCTYPE eagle SYSTEM "eagle.dtd">
-<eagle version="9.1.3">
+<eagle version="9.0.1">
 <drawing>
 <settings>
@@
 <setting verticaltext="up"/>
 </settings>
-<grid distance="50" unitdist="mil" unit="mil" style="lines" multiple="1" display="no" altdistance="5" altunitdist="mil" altunit="mil"/>
+<grid distance="0.1" unitdist="mm" unit="mm" style="dots" multiple="1" display="yes" altdistance="5" altunitdist="mil" altunit="mil"/>
 <layers>
 <layer number="1" name="Top" color="4" fill="1" visible="yes" active="yes"/>
@@
 <param name="checkStop" value="0"/>
 <param name="checkValues" value="0"/>
-<param name="checkNames" value="1"/>
-<param name="checkWireStubs" value="1"/>
-<param name="checkPolygonWidth" value="0"/>
 <param name="useDiameter" value="13"/>
 <param name="maxErrors" value="50"/>
@@
 <signal name="VCC">
 <contactref element="J1" pad="VCC"/>
-<contactref element="U1" pad="5"/>
-<contactref element="C1" pad="2"/>
-<wire x1="3.81" y1="-12.67" x2="3.19" y2="-17.78" width="0" layer="19" extent="1-1"/>
-<wire x1="5.05" y1="-5.89" x2="3.81" y2="-12.67" width="0" layer="19" extent="1-1"/>
 </signal>
 <signal name="GND">
@@
 <wire x1="2.86" y1="-12.67" x2="3.19" y2="-25.4" width="0" layer="19" extent="1-1"/>
 </signal>
+<signal name="N$1">
+<contactref element="U1" pad="5"/>
+<contactref element="C1" pad="2"/>
+<wire x1="3.81" y1="-12.67" x2="3.19" y2="-17.78" width="0" layer="19" extent="1-1"/>
+</signal>
 </signals>
-<mfgpreviewcolors>
-<mfgpreviewcolor name="soldermaskcolor" color="0xC8008000"/>
-<mfgpreviewcolor name="silkscreencolor" color="0xFFFEFEFE"/>
-<mfgpreviewcolor name="backgroundcolor" color="0xFF282828"/>
-<mfgpreviewcolor name="coppercolor" color="0xFFFFBF00"/>
-<mfgpreviewcolor name="substratecolor" color="0xFF786E46"/>
-</mfgpreviewcolors>
 </board>
 </drawing>

Commit message: remove old stuff, make some progress on power
Parts:
- added D1: RED, scono:LED-0603
- added D2: GREEN, scono:LED-0603
- added J2: 2_PIN_JST-XH, scono:2_PIN_JST-XH
- added J3: BL, scono:1X03
- added J4: PWR, scono:1X03
- added J5: UART, scono:1X02
- added R1, R2: 330, scono:R0603
- added R3: 5.1k, scono:R0603
- added U2: AP7312-1833, scono:6-SOT
- U1: value AP7312-1833 -> MCP73831T; device scono:6-SOT -> scono:SOT23-5
- moved U1 16.9 mm to (-10.6, -22.8)
Connections:
- new net MISO: J3.2
- new net MOSI: J3.1
- new net N$2: D2.A, R2.1
- new net N$4: R1.2, R2.2, U1.1
- new net N$5: R3.1, U1.5
- new net RX: J5.1
- new net SCK: J3.3
- new net TX: J5.2
- new net VBAT: C2.2, C3.2, J2.P$2, J4.3, U1.3, U2.3, U2.4, U2.5
- net 1.8V: now also U2.1; no longer C3.2, U1.6
- net 3.3V: now also J4.1, U2.6; no longer C2.2, U1.1, U1.3, U1.4
- net GND: now also D2.C, J2.P$1, J4.2, R3.2, U2.2
- net N$1: now also D1.C, R1.1; no longer C1.2, U1.5
- net VCC: now also C1.2, D1.A, U1.4
Changed lines of the file:
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@@
 <element name="FB1" library="scono" package="0603-FERR" value="" x="2.54" y="-2.54"/>
 <element name="J1" library="scono" package="USB_MICRO" value="USB_MICRO" x="6.35" y="-8.89"/>
-<element name="U1" library="scono" package="6-SOT" value="AP7312-1833" x="3.81" y="-13.97"/>
 <element name="C1" library="scono" package="0402-CAP" value="10uF" x="2.54" y="-17.78">
 <attribute name="PIE-INT-REF-NUM" value="CAPACITOR-GENERIC" x="2.54" y="-17.78" size="1.778" layer="27" display="off"/>
@@
 <attribute name="PIE-INT-REF-NUM" value="CAPACITOR-GENERIC" x="2.54" y="-25.4" size="1.778" layer="27" display="off"/>
 </element>
+<element name="U1" library="scono" package="SOT23-5" value="MCP73831T" x="-10.6" y="-22.8"/>
+<element name="D1" library="scono" package="LED-0603" value="RED" x="-11.1" y="-28.9"/>
+<element name="D2" library="scono" package="LED-0603" value="GREEN" x="-11.1" y="-32.4"/>
+<element name="R1" library="scono" package="R0603" value="330" x="-11.7" y="-36.1">
+<attribute name="DESCRIPTION" value="RESISTOR, American symbol" x="-11.7" y="-36.1" size="1.778" layer="27" display="off"/>
+<attribute name="DISTRIBUTOR" value="DigiKey" x="-11.7" y="-36.1" size="1.778" layer="27" display="off"/>
+<attribute name="DISTRIBUTOR_PART_NUMBER" value="" x="-11.7" y="-36.1" size="1.778" layer="27" display="off"/>
+<attribute name="MANUFACTURER" value="Rohm Semiconductor" x="-11.7" y="-36.1" size="1.778" layer="27" display="off"/>
+<attribute name="MANUFACTURER_PART_NUMBER" value="" x="-11.7" y="-36.1" size="1.778" layer="27" display="off"/>
+<attribute name="NOTES" value="Cut Tape" x="-11.7" y="-36.1" size="1.778" layer="27" display="off"/>
+<attribute name="PACKAGE" value="R0603" x="-11.7" y="-36.1" size="1.778" layer="27" display="off"/>
+</element>
+<element name="R2" library="scono" package="R0603" value="330" x="-11.7" y="-39.8">
+<attribute name="DESCRIPTION" value="RESISTOR, American symbol" x="-11.7" y="-39.8" size="1.778" layer="27" display="off"/>
+<attribute name="DISTRIBUTOR" value="DigiKey" x="-11.7" y="-39.8" size="1.778" layer="27" display="off"/>
+<attribute name="DISTRIBUTOR_PART_NUMBER" value="" x="-11.7" y="-39.8" size="1.778" layer="27" display="off"/>
+<attribute name="MANUFACTURER" value="Rohm Semiconductor" x="-11.7" y="-39.8" size="1.778" layer="27" display="off"/>
+<attribute name="MANUFACTURER_PART_NUMBER" value="" x="-11.7" y="-39.8" size="1.778" layer="27" display="off"/>
+<attribute name="NOTES" value="Cut Tape" x="-11.7" y="-39.8" size="1.778" layer="27" display="off"/>
+<attribute name="PACKAGE" value="R0603" x="-11.7" y="-39.8" size="1.778" layer="27" display="off"/>
+</element>
+<element name="R3" library="scono" package="R0603" value="5.1k" x="-11.7" y="-43.5">
+<attribute name="DESCRIPTION" value="RESISTOR, American symbol" x="-11.7" y="-43.5" size="1.778" layer="27" display="off"/>
+<attribute name="DISTRIBUTOR" value="DigiKey" x="-11.7" y="-43.5" size="1.778" layer="27" display="off"/>
+<attribute name="DISTRIBUTOR_PART_NUMBER" value="" x="-11.7" y="-43.5" size="1.778" layer="27" display="off"/>
+<attribute name="MANUFACTURER" value="Rohm Semiconductor" x="-11.7" y="-43.5" size="1.778" layer="27" display="off"/>
+<attribute name="MANUFACTURER_PART_NUMBER" value="" x="-11.7" y="-43.5" size="1.778" layer="27" display="off"/>
+<attribute name="NOTES" value="Cut Tape" x="-11.7" y="-43.5" size="1.778" layer="27" display="off"/>
+<attribute name="PACKAGE" value="R0603" x="-11.7" y="-43.5" size="1.778" layer="27" display="off"/>
+</element>
+<element name="U2" library="scono" package="6-SOT" value="AP7312-1833" x="-16.7" y="-42.2"/>
+<element name="J2" library="scono" package="2_PIN_JST-XH" value="2_PIN_JST-XH" x="-14.4" y="-56.3"/>
+<element name="J4" library="scono" package="1X03" package3d_urn="urn:adsk.eagle:package:38063/1" value="PWR" x="-10.1" y="-88.7"/>
+<element name="J3" library="scono" package="1X03" package3d_urn="urn:adsk.eagle:package:38063/1" value="BL" x="-10.1" y="-107.5"/>
+<element name="J5" library="scono" package="1X02" package3d_urn="urn:adsk.eagle:package:38039/1" value="UART" x="-10.1" y="-126.3"/>
 </elements>
 <signals>
 <signal name="VCC">
 <contactref element="J1" pad="VCC"/>
+<contactref element="C1" pad="2"/>
+<contactref element="U1" pad="4"/>
+<contactref element="D1" pad="A"/>
+<wire x1="-9.65" y1="-21.5" x2="-11.977" y2="-28.9" width="0" layer="19" extent="1-1"/>
+<wire x1="3.19" y1="-17.78" x2="-9.65" y2="-21.5" width="0" layer="19" extent="1-1"/>
+<wire x1="5.05" y1="-5.89" x2="3.19" y2="-17.78" width="0" layer="19" extent="1-1"/>
 </signal>
 <signal name="GND">
@@
 <contactref element="FB1" pad="1"/>
 <contactref element="C1" pad="1"/>
-<contactref element="U1" pad="2"/>
 <contactref element="C2" pad="1"/>
 <contactref element="C3" pad="1"/>
+<contactref element="D2" pad="C"/>
+<contactref element="U1" pad="2"/>
+<contactref element="R3" pad="2"/>
+<contactref element="U2" pad="2"/>
+<contactref element="J2" pad="P$1"/>
+<contactref element="J4" pad="2"/>
+<wire x1="-11.95" y1="-52.9" x2="-7.56" y2="-88.7" width="0" layer="19" extent="1-1"/>
+<wire x1="-10.85" y1="-43.5" x2="-11.95" y2="-52.9" width="0" layer="19" extent="1-1"/>
+<wire x1="-16.7" y1="-43.5" x2="-10.85" y2="-43.5" width="0" layer="19" extent="1-1"/>
+<wire x1="-10.223" y1="-32.4" x2="-10.85" y2="-43.5" width="0" layer="19" extent="1-1"/>
+<wire x1="-10.6" y1="-24.09" x2="-10.223" y2="-32.4" width="0" layer="19" extent="1-1"/>
+<wire x1="1.89" y1="-25.4" x2="-10.6" y2="-24.09" width="0" layer="19" extent="1-1"/>
 <wire x1="1.89" y1="-21.59" x2="1.89" y2="-25.4" width="0" layer="19" extent="1-1"/>
 <wire x1="1.89" y1="-17.78" x2="1.89" y2="-21.59" width="0" layer="19" extent="1-1"/>
-<wire x1="3.81" y1="-15.27" x2="1.89" y2="-17.78" width="0" layer="19" extent="1-1"/>
-<wire x1="7.65" y1="-5.89" x2="3.81" y2="-15.27" width="0" layer="19" extent="1-1"/>
+<wire x1="7.65" y1="-5.89" x2="1.89" y2="-17.78" width="0" layer="19" extent="1-1"/>
 <wire x1="1.69" y1="-2.54" x2="7.65" y2="-5.89" width="0" layer="19" extent="1-1"/>
 </signal>
@@
 <contactref element="FB1" pad="2"/>
 </signal>
-<signal name="3.3V">
-<contactref element="U1" pad="4"/>
+<signal name="N$1">
+<contactref element="D1" pad="C"/>
+<contactref element="R1" pad="1"/>
+<wire x1="-10.223" y1="-28.9" x2="-12.55" y2="-36.1" width="0" layer="19" extent="1-1"/>
+</signal>
+<signal name="N$2">
+<contactref element="R2" pad="1"/>
+<contactref element="D2" pad="A"/>
+<wire x1="-11.977" y1="-32.4" x2="-12.55" y2="-39.8" width="0" layer="19" extent="1-1"/>
+</signal>
+<signal name="N$4">
+<contactref element="R1" pad="2"/>
+<contactref element="U1" pad="1"/>
+<contactref element="R2" pad="2"/>
+<wire x1="-10.85" y1="-36.1" x2="-10.85" y2="-39.8" width="0" layer="19" extent="1-1"/>
+<wire x1="-11.55" y1="-24.09" x2="-10.85" y2="-36.1" width="0" layer="19" extent="1-1"/>
+</signal>
+<signal name="N$5">
+<contactref element="U1" pad="5"/>
+<contactref element="R3" pad="1"/>
+<wire x1="-11.55" y1="-21.5" x2="-12.55" y2="-43.5" width="0" layer="19" extent="1-1"/>
+</signal>
+<signal name="VBAT">
 <contactref element="U1" pad="3"/>
 <contactref element="C2" pad="2"/>
-<contactref element="U1" pad="1"/>
-<wire x1="2.86" y1="-15.27" x2="3.19" y2="-21.59" width="0" layer="19" extent="1-1"/>
-<wire x1="4.76" y1="-15.27" x2="2.86" y2="-15.27" width="0" layer="19" extent="1-1"/>
-<wire x1="4.76" y1="-12.67" x2="4.76" y2="-15.27" width="0" layer="19" extent="1-1"/>
+<contactref element="U2" pad="5"/>
+<contactref element="U2" pad="4"/>
+<contactref element="U2" pad="3"/>
+<contactref element="J2" pad="P$2"/>
+<contactref element="C3" pad="2"/>
+<contactref element="J4" pad="3"/>
+<wire x1="-9.45" y1="-52.9" x2="-5.02" y2="-88.7" width="0" layer="19" extent="1-1"/>
+<wire x1="-15.75" y1="-43.5" x2="-9.45" y2="-52.9" width="0" layer="19" extent="1-1"/>
+<wire x1="-15.75" y1="-40.9" x2="-15.75" y2="-43.5" width="0" layer="19" extent="1-1"/>
+<wire x1="-16.7" y1="-40.9" x2="-15.75" y2="-40.9" width="0" layer="19" extent="1-1"/>
+<wire x1="-9.65" y1="-24.09" x2="-15.75" y2="-40.9" width="0" layer="19" extent="1-1"/>
+<wire x1="3.19" y1="-25.4" x2="-9.65" y2="-24.09" width="0" layer="19" extent="1-1"/>
+<wire x1="3.19" y1="-21.59" x2="3.19" y2="-25.4" width="0" layer="19" extent="1-1"/>
 </signal>
 <signal name="1.8V">
-<contactref element="C3" pad="2"/>
-<contactref element="U1" pad="6"/>
-<wire x1="2.86" y1="-12.67" x2="3.19" y2="-25.4" width="0" layer="19" extent="1-1"/>
+<contactref element="U2" pad="1"/>
 </signal>
-<signal name="N$1">
-<contactref element="U1" pad="5"/>
-<contactref element="C1" pad="2"/>
-<wire x1="3.81" y1="-12.67" x2="3.19" y2="-17.78" width="0" layer="19" extent="1-1"/>
+<signal name="3.3V">
+<contactref element="U2" pad="6"/>
+<contactref element="J4" pad="1"/>
+<wire x1="-17.65" y1="-40.9" x2="-10.1" y2="-88.7" width="0" layer="19" extent="1-1"/>
+</signal>
+<signal name="SCK">
+<contactref element="J3" pad="3"/>
+</signal>
+<signal name="MISO">
+<contactref element="J3" pad="2"/>
+</signal>
+<signal name="MOSI">
+<contactref element="J3" pad="1"/>
+</signal>
+<signal name="TX">
+<contactref element="J5" pad="2"/>
+</signal>
+<signal name="RX">
+<contactref element="J5" pad="1"/>
 </signal>
 </signals>
 </board>
 </drawing>
+<compatibility>
+<note version="8.3" severity="warning">
+Since Version 8.3, EAGLE supports URNs for individual library
+assets (packages, symbols, and devices). The URNs of those assets
+will not be understood (or retained) with this version.
+</note>
+<note version="8.3" severity="warning">
+Since Version 8.3, EAGLE supports the association of 3D packages
+with devices in libraries, schematics, and board files. Those 3D
+packages will not be understood (or retained) with this version.
+</note>
+</compatibility>
 </eagle>

Commit message: do more audio stuff
Parts:
- added C10: 1uF, scono:0603-CAP
- added C11, C15, C19: 10uF, scono:0402-CAP
- added C12, C13, C14, C16, C17, C18, C20, C21, C22: 0.1uF, scono:0402-CAP
- added C4: (no value), scono:0603-CAP
- added C5, C6: 18pF, scono:0603-CAP
- added C7, C8: 10nF, scono:0603-CAP
- added C9: 47nF, scono:0603-CAP
- added FB2: (no value), scono:0603-FERR
- added R10, R4: 100K, scono:R0603
- added R11: 1M, scono:R0603
- added R5: 10R, scono:R0603
- added R6, R7: >VALUE, scono:R0603
- added R8, R9: 20R, scono:R0603
- added U3: VS1053, scono:QFP50P900X900X120-48N
- added U4: ATMEGA328PB-AUR, scono:QFP80P900X900X120-32N
- added Y1: ABM8G-12.288MHZ-18-D2Y-T, scono:OSCSC320X250X100N
- R1, R2: value 330 -> 330R
- R3: value 5.1k -> 10k
- moved J5 238.8 mm to (0.70, 112.3)
Connections:
- new net AVCC: U4.18
- new net AVDD: C11.2, C12.2, C13.2, C14.2, FB2.1, U3.38, U3.43, U3.45
- new net DREG: U3.8
- new net GBUF: R5.1, U3.42
- new net LEFT: R9.1, U3.46
- new net N$23: U3.15
- new net N$24: C9.2, R5.2
- new net N$25: C8.1, R9.2
- new net N$27: R10.1, U3.10, U3.11, U3.12, U3.25, U3.33, U3.34, U3.36, U3.9
- new net N$3: C7.2, R8.2
- new net N$7: C4.2, R4.2, U3.3
- new net RCAP: C10.2, U3.44
- new net RIGHT: R8.1, U3.39
- new net SCLK: U3.28
- new net VSCS: U3.23
- new net VSDCS: U3.13
- new net XTALIN: C5.1, R11.2, U3.18, Y1.3
- new net XTALOUT: C6.1, R11.1, U3.17, Y1.1
- net 1.8V: now also C19.2, C20.2, C21.2, C22.2, U3.24, U3.31, U3.5, U3.7
- net 3.3V: now also C15.2, C16.2, C17.2, C18.2, FB2.2, R4.1, U3.14, U3.19, U3.26, U3.32, U3.6, U4.4
- net AGND: now also C10.1, C11.1, C12.1, C13.1, C14.1, C7.1, C8.2, C9.1, U3.37, U3.40, U3.41, U3.47
- net GND: now also C15.1, C16.1, C17.1, C18.1, C19.1, C20.1, C21.1, C22.1, C4.1, C5.2, C6.2, R10.2, U3.16, U3.20, U3.21, U3.22, U3.35, U3.4, U4.21, U4.5, Y1.2, Y1.4
- net MISO: now also U3.30
- net MOSI: now also U3.29

Commit message: do more work on schem - need to add microphone
Parts:
- removed R7: >VALUE, scono:R0603
- added C23, C24: 18pF, scono:0603-CAP
- added P1: MICROSD, scono:MICROSD
- added R12: 1M, scono:R0603
- added Y2: 8MHz, scono:XTAL500X320X130N
- J5: value UART -> FLASH; device scono:1X02 -> scono:1X03
- R6: value >VALUE -> 10K
- moved J5 251.1 mm to (-35.7, -136.1)
- moved R6 241.3 mm to (-43.2, -147.4)
Connections:
- removed net DREG: U3.8
- removed net N$7: C4.2, R4.2, U3.3
- removed net VSDCS: U3.13
- new net DREQ: U3.8, U4.1
- new net N$6: C23.2, R12.1, U4.7, Y2.1
- new net N$8: C24.2, R12.2, U4.8, Y2.2
- new net RST: J5.1, R6.2, U4.29
- new net SDCS: P1.2, U4.2
- new net VSRST: C4.2, R4.2, U3.3, U4.13
- new net XDCS: U3.13, U4.12
- net 3.3V: now also P1.4, R6.1
- net GND: now also C23.1, C24.1, P1.6
- net MISO: now also P1.7, U4.16
- net MOSI: now also P1.3, U4.15
- net RX: now also J5.2, U4.30; no longer J5.1
- net SCK: now also P1.5, U4.17
- net TX: now also J5.3, U4.31; no longer J5.2
- net VSCS: now also U4.14

Commit message: left over commit
Parts:
- added J6: SJ-3524-SMT, scono:CUI_SJ-3524-SMT
- added R13, R14, R7: 100k, scono:R0603
Connections:
- new net N$10: J6.4
- new net N$11: R14.2, U4.9
- new net N$7: R7.2, U4.11
- new net N$9: R13.2, U4.10
- net GND: now also J6.1, R13.1, R14.1, R7.1
- net LEFT: now also J6.2
- net RIGHT: now also J6.3
Changed lines of the file:
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@@
 </element>
 <element name="P1" library="scono" package="MICROSD" value="MICROSD" x="-53.3" y="-142.3"/>
+<element name="J6" library="scono" package="CUI_SJ-3524-SMT" value="SJ-3524-SMT" x="-53.9" y="-157.6">
+<attribute name="CUI_PURCHASE_URL" value="https://www.cui.com/product/interconnect/audio-connectors/3.5-mm-jacks/sj-352x-smt-series?utm_source=snapeda.com&amp;utm_medium=referral&amp;utm_campaign=snapedaBOM" x="-53.9" y="-157.6" size="1.778" layer="27" display="off"/>
+<attribute name="DESCRIPTION" value=" SJ Series 3.5 mm 12 V SMT Right Angle Stereo Audio Jack " x="-53.9" y="-157.6" size="1.778" layer="27" display="off"/>
+<attribute name="DIGI-KEY_PART_NUMBER" value="CP-3524SJCT-ND" x="-53.9" y="-157.6" size="1.778" layer="27" display="off"/>
+<attribute name="DIGI-KEY_PURCHASE_URL" value="https://www.digikey.com/product-detail/en/cui-inc/SJ-3524-SMT-TR/CP-3524SJCT-ND/669705?utm_source=snapeda&amp;utm_medium=aggregator&amp;utm_campaign=symbol" x="-53.9" y="-157.6" size="1.778" layer="27" display="off"/>
+<attribute name="MF" value="CUI Inc." x="-53.9" y="-157.6" size="1.778" layer="27" display="off"/>
+<attribute name="MP" value="SJ-3524-SMT-TR" x="-53.9" y="-157.6" size="1.778" layer="27" display="off"/>
+<attribute name="PACKAGE" value="None" x="-53.9" y="-157.6" size="1.778" layer="27" display="off"/>
+</element>
+<element name="R7" library="scono" package="R0603" value="100k" x="-58.2" y="-167.8">
+<attribute name="DESCRIPTION" value="RESISTOR, American symbol" x="-58.2" y="-167.8" size="1.778" layer="27" display="off"/>
+<attribute name="DISTRIBUTOR" value="DigiKey" x="-58.2" y="-167.8" size="1.778" layer="27" display="off"/>
+<attribute name="DISTRIBUTOR_PART_NUMBER" value="" x="-58.2" y="-167.8" size="1.778" layer="27" display="off"/>
+<attribute name="MANUFACTURER" value="Rohm Semiconductor" x="-58.2" y="-167.8" size="1.778" layer="27" display="off"/>
+<attribute name="MANUFACTURER_PART_NUMBER" value="" x="-58.2" y="-167.8" size="1.778" layer="27" display="off"/>
+<attribute name="NOTES" value="Cut Tape" x="-58.2" y="-167.8" size="1.778" layer="27" display="off"/>
+<attribute name="PACKAGE" value="R0603" x="-58.2" y="-167.8" size="1.778" layer="27" display="off"/>
+</element>
+<element name="R13" library="scono" package="R0603" value="100k" x="-58.2" y="-171.5">
+<attribute name="DESCRIPTION" value="RESISTOR, American symbol" x="-58.2" y="-171.5" size="1.778" layer="27" display="off"/>
+<attribute name="DISTRIBUTOR" value="DigiKey" x="-58.2" y="-171.5" size="1.778" layer="27" display="off"/>
+<attribute name="DISTRIBUTOR_PART_NUMBER" value="" x="-58.2" y="-171.5" size="1.778" layer="27" display="off"/>
+<attribute name="MANUFACTURER" value="Rohm Semiconductor" x="-58.2" y="-171.5" size="1.778" layer="27" display="off"/>
+<attribute name="MANUFACTURER_PART_NUMBER" value="" x="-58.2" y="-171.5" size="1.778" layer="27" display="off"/>
+<attribute name="NOTES" value="Cut Tape" x="-58.2" y="-171.5" size="1.778" layer="27" display="off"/>
+<attribute name="PACKAGE" value="R0603" x="-58.2" y="-171.5" size="1.778" layer="27" display="off"/>
+</element>
+<element name="R14" library="scono" package="R0603" value="100k" x="-58.2" y="-175.2">
+<attribute name="DESCRIPTION" value="RESISTOR, American symbol" x="-58.2" y="-175.2" size="1.778" layer="27" display="off"/>
+<attribute name="DISTRIBUTOR" value="DigiKey" x="-58.2" y="-175.2" size="1.778" layer="27" display="off"/>
+<attribute name="DISTRIBUTOR_PART_NUMBER" value="" x="-58.2" y="-175.2" size="1.778" layer="27" display="off"/>
+<attribute name="MANUFACTURER" value="Rohm Semiconductor" x="-58.2" y="-175.2" size="1.778" layer="27" display="off"/>
+<attribute name="MANUFACTURER_PART_NUMBER" value="" x="-58.2" y="-175.2" size="1.778" layer="27" display="off"/>
+<attribute name="NOTES" value="Cut Tape" x="-58.2" y="-175.2" size="1.778" layer="27" display="off"/>
+<attribute name="PACKAGE" value="R0603" x="-58.2" y="-175.2" size="1.778" layer="27" display="off"/>
+</element>
 </elements>
 <signals>
@@
 <contactref element="C23" pad="1"/>
 <contactref element="P1" pad="6"/>
+<contactref element="J6" pad="1"/>
+<contactref element="R7" pad="1"/>
+<contactref element="R13" pad="1"/>
+<contactref element="R14" pad="1"/>
+<wire x1="-59.05" y1="-171.5" x2="-59.05" y2="-175.2" width="0" layer="19" extent="1-1"/>
+<wire x1="-59.05" y1="-167.8" x2="-59.05" y2="-171.5" width="0" layer="19" extent="1-1"/>
+<wire x1="-55" y1="-161.3" x2="-59.05" y2="-167.8" width="0" layer="19" extent="1-1"/>
+<wire x1="-55.6995" y1="-142.05" x2="-55" y2="-161.3" width="0" layer="19" extent="1-1"/>
 <wire x1="-43.25" y1="-121" x2="-55.6995" y2="-142.05" width="0" layer="19" extent="1-1"/>
 <wire x1="-43.25" y1="-118.4" x2="-43.25" y2="-121" width="0" layer="19" extent="1-1"/>
@@
 <contactref element="U3" pad="46"/>
 <contactref element="R9" pad="1"/>
+<contactref element="J6" pad="2"/>
+<wire x1="-33.05" y1="66.9" x2="-45.6" y2="-161.3" width="0" layer="19" extent="1-1"/>
 <wire x1="-16.9526" y1="115.4164" x2="-33.05" y2="66.9" width="0" layer="19" extent="1-1"/>
 </signal>
@@
 <contactref element="U3" pad="39"/>
 <contactref element="R8" pad="1"/>
+<contactref element="J6" pad="3"/>
+<wire x1="-33.05" y1="70.6" x2="-53" y2="-153.9" width="0" layer="19" extent="1-1"/>
 <wire x1="-13.4474" y1="115.4164" x2="-33.05" y2="70.6" width="0" layer="19" extent="1-1"/>
 </signal>
@@
 <wire x1="-31.67" y1="112.4" x2="-19.4164" y2="110.438" width="0" layer="19" extent="1-1"/>
 </signal>
+<signal name="N$10">
+<contactref element="J6" pad="4"/>
+</signal>
+<signal name="N$7">
+<contactref element="U4" pad="11"/>
+<contactref element="R7" pad="2"/>
+<wire x1="-28.7" y1="105.43" x2="-57.35" y2="-167.8" width="0" layer="19" extent="1-1"/>
+</signal>
+<signal name="N$9">
+<contactref element="U4" pad="10"/>
+<contactref element="R13" pad="2"/>
+<wire x1="-29.5" y1="105.43" x2="-57.35" y2="-171.5" width="0" layer="19" extent="1-1"/>
+</signal>
+<signal name="N$11">
+<contactref element="U4" pad="9"/>
+<contactref element="R14" pad="2"/>
+<wire x1="-30.3" y1="105.43" x2="-57.35" y2="-175.2" width="0" layer="19" extent="1-1"/>
+</signal>
 </signals>
